File: example/DA26R_DA30R.kicad_pcb (KiCad board)
At the start: 4 copper layers, 95.9 x 20 mm, 202 parts, among them J1 PWR, J10 Sensor, J11 HALL, J12 Conn_JST_B3B_EH_01x03, J13 RS485, J2 SW, J3 INT, J4 Sensor, J5 HALL, J6 Conn_JST_B3B_EH_01x03, J7 PWR, J8 SW, J9 INT, U1 INA194, U10 DRV8320S, U11 TLP3412, U12 INA194, U13 MIC6270, U14 ATSAMC21G18A-MNT, U15 MAX15062BATA+T, U16 THVD2410DRBR, U17 THVD2410DRBR, U18 TLP3412, U19 THVD2410DRBR, U2 MIC6270, U20 MCP2542FDT, U21 DRV8320S, U22 TLP3412, U3 ATSAMC21G18A-MNT, U4 MAX15062BATA+T, U5 THVD2410DRBR, U6 THVD2410DRBR, U7 TLP3412, U8 THVD2410DRBR, U9 MCP2542FDT

Commit message: Rebuilding code to unify regexps, doesn't work yet
Parts:
- removed the C64 at (242.3, 56.3)
- removed the C64 at (259.1, 35.9)
- removed the R54 at (257.3, 43.2)
- added C64: 1.0, VolzLib:C0603, F.Cu at (239.3, 29.0)
- moved J7 41.4 mm to (192.7, 35.9)
- moved J9 41.4 mm to (184.9, 38.2)
- moved R51 0.73 mm to (257.9, 46.0)
Connections:
- net +28V1 renamed /ACE1/+28V
- net +28V2 renamed /ACE2/+28V
- net +5V1 renamed /ACE1/+5V
- net +ARM1 renamed /ACE1/+ARM
- net +ARM2 renamed /ACE2/+ARM
- net /ACE1/A1 renamed /ACE1/RS_A
- net /ACE1/B1 renamed /ACE1/RS_B
- net /ACE1/BRAKE1 renamed /ACE1/BRAKE
- net /ACE1/CANH1 renamed /ACE1/CANH
- net /ACE1/CANL1 renamed /ACE1/CANL
- net /ACE1/CAN_R1 renamed /ACE1/CAN_R
- net /ACE1/CAN_T1 renamed /ACE1/CAN_T
- net /ACE1/CURR1 renamed /ACE1/CURR
- net /ACE1/CURRL1 renamed /ACE1/CURRL
- net /ACE1/DCI1 renamed /ACE1/DCI
- net /ACE1/DCIN1 renamed /ACE1/DCIN
- net /ACE1/DCO1 renamed /ACE1/DCO
- net /ACE1/DCOUT1 renamed /ACE1/DCOUT
- net /ACE1/DIR_EXT1 renamed /ACE1/DIR_EXT
- net /ACE1/DIR_INT1 renamed /ACE1/DIR_INT
- net /ACE1/HA1 renamed Net-(J5-Pad3)
- net /ACE1/HB1 renamed Net-(J5-Pad4)
- net /ACE1/HC1 renamed Net-(J5-Pad5)
- net /ACE1/H_A1 renamed /ACE1/H_A
- net /ACE1/H_B1 renamed /ACE1/H_B
- net /ACE1/H_C1 renamed /ACE1/H_C
- net /ACE1/MEN1 renamed /ACE1/MEN
- net /ACE1/MISO1 renamed /ACE1/MISO
- net /ACE1/MOSI1 renamed /ACE1/MOSI
- net /ACE1/MOT_DIR1 renamed /ACE1/MOT_DIR
- net /ACE1/MOT_EN1 renamed /ACE1/MOT_EN
- net /ACE1/MOT_T1 renamed /ACE1/MOT_T
- net /ACE1/MSCS1 renamed /ACE1/MSCS
- net /ACE1/OPTO_A1 renamed /ACE1/OPTO_A
- net /ACE1/OPTO_C1 renamed /ACE1/OPTO_C
- net /ACE1/PHASE_A1 renamed /ACE1/PHASE_A
- net /ACE1/PHASE_B1 renamed /ACE1/PHASE_B
- net /ACE1/PHASE_C1 renamed /ACE1/PHASE_C
- net /ACE1/PWM1 renamed /ACE1/PWM
- net /ACE1/RST1 renamed /ACE1/RST
- net /ACE1/RX_EXT1 renamed /ACE1/RX_EXT
- net /ACE1/RX_INT1 renamed /ACE1/RX_INT
- net /ACE1/SCLK1 renamed /ACE1/SCLK
- net /ACE1/SCS1 renamed /ACE1/SCS
- net /ACE1/SWC1 renamed /ACE1/SWC
- net /ACE1/SWD1 renamed /ACE1/SWD
- net /ACE1/TE1 renamed /ACE1/TE
- net /ACE1/TX_EXT1 renamed /ACE1/TX_EXT
- net /ACE1/TX_INT1 renamed /ACE1/TX_INT
- net /ACE1/U5V1 renamed /ACE1/U5V
- net /ACE1/VOLTP1 renamed /ACE1/VOLTP
- net /ACE1/VOLTS1 renamed /ACE1/VOLTS
- net /ACE1/Y1 renamed /ACE1/RS_Y
- net /ACE1/Z1 renamed /ACE1/RS_Z
- net /ACE2/A2 renamed /ACE2/RS_A
- net /ACE2/B2 renamed /ACE2/RS_B
- net /ACE2/BRAKE2 renamed /ACE2/BRAKE
- net /ACE2/CANH2 renamed /ACE2/CANH
- net /ACE2/CANL2 renamed /ACE2/CANL
- net /ACE2/CAN_R2 renamed /ACE2/CAN_R
- net /ACE2/CAN_T2 renamed /ACE2/CAN_T
- net /ACE2/CURR2 renamed /ACE2/CURR
- net /ACE2/CURRL2 renamed /ACE2/CURRL
- net /ACE2/DCI2 renamed /ACE2/DCI
- net /ACE2/DCIN2 renamed /ACE2/DCIN
- net /ACE2/DCO2 renamed /ACE2/DCO
- net /ACE2/DCOUT2 renamed /ACE2/DCOUT
- net /ACE2/DIR_EXT2 renamed /ACE2/DIR_EXT
- net /ACE2/DIR_INT2 renamed /ACE2/DIR_INT
- net /ACE2/HA2 renamed Net-(J11-Pad3)
- net /ACE2/HB2 renamed Net-(J11-Pad4)
- net /ACE2/HC2 renamed Net-(J11-Pad5)
- net /ACE2/H_A2 renamed /ACE2/H_A
- net /ACE2/H_B2 renamed /ACE2/H_B
- net /ACE2/H_C2 renamed /ACE2/H_C
- net /ACE2/MEN2 renamed /ACE2/MEN
- net /ACE2/MISO2 renamed /ACE2/MISO
- net /ACE2/MOSI2 renamed /ACE2/MOSI
- net /ACE2/MOT_DIR2 renamed /ACE2/MOT_DIR
- net /ACE2/MOT_EN2 renamed /ACE2/MOT_EN
- net /ACE2/MOT_T2 renamed /ACE2/MOT_T
- net /ACE2/MSCS2 renamed /ACE2/MSCS
- net /ACE2/OPTO_A2 renamed /ACE2/OPTO_A
- net /ACE2/OPTO_C2 renamed /ACE2/OPTO_C
- net /ACE2/PHASE_A2 renamed /ACE2/PHASE_A
- net /ACE2/PHASE_B2 renamed /ACE2/PHASE_B
- net /ACE2/PHASE_C2 renamed /ACE2/PHASE_C
- net /ACE2/PWM2 renamed /ACE2/PWM
- net /ACE2/RST2 renamed /ACE2/RST
- net /ACE2/RX_EXT2 renamed /ACE2/RX_EXT
- net /ACE2/RX_INT2 renamed /ACE2/RX_INT
- net /ACE2/SCLK2 renamed /ACE2/SCLK
- net /ACE2/SWC2 renamed /ACE2/SWC
- net /ACE2/SWD2 renamed /ACE2/SWD
- net /ACE2/TE2 renamed /ACE2/TE
- net /ACE2/TX_EXT2 renamed /ACE2/TX_EXT
- net /ACE2/TX_INT2 renamed /ACE2/TX_INT
- net /ACE2/U5V2 renamed /ACE2/U5V
- net /ACE2/VOLTP2 renamed /ACE2/VOLTP
- net /ACE2/VOLTS2 renamed /ACE2/VOLTS
- net /ACE2/Y2 renamed /ACE2/RS_Y
- net /ACE2/Z2 renamed /ACE2/RS_Z
- C38 pad 1: +5V2 -> /ACE2/+5V
- C42 pad 1: +5V2 -> /ACE2/+5V
- C52 pad 1: +5V2 -> /ACE2/+5V
- C55 pad 1: +5V2 -> /ACE2/+5V
- C56 pad 1: +5V2 -> /ACE2/+5V
- C57 pad 1: +5V2 -> /ACE2/+5V
- C58 pad 1: +5V2 -> /ACE2/+5V
- C59 pad 1: +5V2 -> /ACE2/+5V
- D10 pad 2: +5V2 -> /ACE2/+5V
- D11 pad 2: +5V2 -> /ACE2/+5V
- D9 pad 2: +5V2 -> /ACE2/+5V
- J10 pad 1: +5V2 -> /ACE2/+5V
- J10 pad 7: +5V2 -> /ACE2/+5V
- J11 pad 1: +5V2 -> /ACE2/+5V
- L4 pad 2: +5V2 -> /ACE2/+5V
- R34 pad 1: +5V2 -> /ACE2/+5V
- R40 pad 2: +5V2 -> /ACE2/+5V
- R42 pad 1: +5V2 -> /ACE2/+5V
- U12 pad 5: +5V2 -> /ACE2/+5V
- U13 pad 5: +5V2 -> /ACE2/+5V
- U14 pad 32: /ACE2/SCS2 -> /ACE2/SCS
- U15 pad 4: +5V2 -> /ACE2/+5V
- U16 pad 8: +5V2 -> /ACE2/+5V
- U17 pad 8: +5V2 -> /ACE2/+5V
- U19 pad 8: +5V2 -> /ACE2/+5V
- U20 pad 3: +5V2 -> /ACE2/+5V
- U20 pad 5: +5V2 -> /ACE2/+5V
Routing:
- added copper zone on In2.Cu, net +28V1
- removed copper zone on In2.Cu, net /ACE1/+28V
